File: hardware/0.2/mini4wd-motor-tester.kicad_sch (KiCad schematic)
At the start: 114 parts, among them J1 USB_C_Receptacle_USB2.0_16P, J2 JST SH, J4 JST XH, M1 Motor_DC, M2 TP, M3 TP, Q2 AO3401A, Q3 2N7002, SW1 RA, SW2 RA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

Commit message: add v2 heatsink, improve layout for v2 main
Parts:
- added C26, C27: 10u, Capacitor_SMD:C_0805_2012Metric, symbol Device:C
- renumbered M3 to M2, M2 to M3
Connections:
- net +5V: now also C27.1
- net GND: now also C26.2, C27.2
- net at C17.1, C23.1, R13.2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: now also C26.1
Other:
- moved on the sheet: C3, C4, FB1

Commit message: minor sch and pcb updates
Parts:
- J4: LCSC (none) -> C157931; MPN  (none) -> S2B-XH-A(LF)(SN)
- R16: LCSC (none) -> C23186; MPN  (none) -> 0603WAF5101T5E
- R17, R25: LCSC (none) -> C8218; MPN  (none) -> 0603WAF2000T5E
- R22, R26: LCSC (none) -> C25819; MPN  (none) -> 0603WAF4702T5E
- R29, R32: value 180K -> 200K; LCSC (none) -> C25811; MPN  (none) -> 0603WAF2003T5E; Manufacturer (none) -> UNI-ROYAL
- R7: LCSC (none) -> C25803; MPN  (none) -> 0603WAF1003T5E
- R8: LCSC (none) -> C4216; MPN  (none) -> 0603WAF3302T5E
- RV1, RV2: LCSC (none) -> C719186
- U11, U13: LCSC (none) -> C702117; MPN  (none) -> TLV7011DBVR; Manufacturer (none) -> TI
Connections:
- net +5V: no longer U2.5 (VBUS)
- net at C5.1, F1.2, FB2.2: now also U2.5 (VBUS)
Other:
- moved on the sheet: C10, C13, C14, C5, C6, C7, D1, D2, FB2, J2, R10, R12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

Commit message: off to fab
Changed lines of the file:
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@@
+		)
+	)
+	(text_box "VREF set by RV2, default VCC/2\nHysteresis = +/- 185mV\n\nTIDU020, Section 2.1\nRh/Rx = 1.465/(1.835-1.465) = 4\nRy/Rx = 1.465/(3.3-1.835) = 1\nRx = 50K, Rh = 200K"
+		(exclude_from_sim no)
+		(at 363.22 146.05 0)
+		(size 39.37 15.24)
+		(margins 0.9525 0.9525 0.9525 0.9525)
+		(stroke
+			(width -0.0001)
+			(type solid)
+		)
+		(fill
+			(type none)
+		)
+		(effects
+			(font
+				(size 1.27 1.27)
+				(thickness 0.254)
+				(bold yes)
+			)
+			(justify left top)
 		)
 	)
@@
 		)
 	)
-	(text_box "VREF set by RV2, default VCC/2\nHysteresis = +/- 175mV\n\nTIDU020, Section 2.1\nRh/Rx = 1.475/(1.825-1.475) = 4.2\nRy/Rx = 1.475/(3.3-1.825) = 1\nRx = 50K, Rh = 210.7K"
-		(exclude_from_sim no)
-		(at 363.22 147.32 0)
-		(size 39.37 15.24)
-		(margins 0.9525 0.9525 0.9525 0.9525)
-		(stroke
-			(width -0.0001)
-			(type solid)
-		)
-		(fill
-			(type none)
-		)
-		(effects
-			(font
-				(size 1.27 1.27)
-				(thickness 0.254)
-				(bold yes)
-			)
-			(justify left top)
-		)
-	)
 	(text_box "IMAX = 2A\nRshunt = 10mR\nVdrop = 20mV (< 40mV FS)\nP = 2^2 * 10m\n  = 40mW"
 		(exclude_from_sim no)
@@
 		)
 	)
-	(text_box "VREF set by RV2, default VCC/2\nHysteresis = +/- 175mV\n\nTIDU020, Section 2.1\nRh/Rx = 1.475/(1.825-1.475) = 4.2\nRy/Rx = 1.475/(3.3-1.825) = 1\nRx = 50K, Rh = 210.7K"
+	(text_box "VREF set by RV2, default VCC/2\nHysteresis = +/- 185mV\n\nTIDU020, Section 2.1\nRh/Rx = 1.465/(1.835-1.465) = 4\nRy/Rx = 1.465/(3.3-1.835) = 1\nRx = 50K, Rh = 200K"
 		(exclude_from_sim no)
 		(at 67.31 262.89 0)
